File: KiCad_files/WatchPad_2layer.kicad_sch (KiCad schematic)
At the start: 44 parts, among them SW1 SW_Push, SW10 SW_Push, SW11 SW_Push, SW12 SW_Push, SW2 SW_Push, SW3 SW_Push, SW4 SW_Push, SW5 SW_Push, SW6 SW_Push, SW7 SW_Push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

Commit message: Added BOM and Slightly changed PCB layout
Changed mounting solution for speaker to use more standard 6.5mm hole spacing
Parts:
- LS1: footprint Buzzer_Beeper:Buzzer_12x9.5RM7.6 -> Buzzer_Beeper:Buzzer_TDK_PS1240P02BT_D12.2mm_H6.5mm
Changed lines of the file:
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@@
 			)
 		)
-		(property "Footprint" "Buzzer_Beeper:Buzzer_12x9.5RM7.6"
+		(property "Footprint" "Buzzer_Beeper:Buzzer_TDK_PS1240P02BT_D12.2mm_H6.5mm"
 			(at 25.4 57.15 0)
 			(effects
